File: hardware/paddle-bridge/paddle_bridge.kicad_sch (KiCad schematic)
At the start: 15 parts, among them J1 APOLLO (P4 header GND,52,51,5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, J2 MACHINE: paddle pair + Micra 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, U1 AQY212EH, U2 LH1502BB, U3 LH1502BB

Commit message: hardware: Apollo Link rev 0.6 - USB-C 5 V in, powers the Apollo over J1; gerbers + BOM
The bridge now carries a 5 V rail so a single 5-conductor cable can power
the remote through the P4's 40-pin header instead of a second USB lead:

- J3: GCT USB4085-GF-A USB-C receptacle (THT), power only. R9/R10 5k1 Rd
  on CC1/CC2 so any USB-C source, PD or not, turns VBUS on at 5 V.
- F1: 1.5 A hold / 3 A trip PTC (Littelfuse 1812L150/12DR) between VBUS
  and the 5V net; the Apollo peaks at ~0.6 A, and the hold current still
  clears that at the 85 C in-chassis limit. VBUS/5V tracks 0.5 mm.
- J1 grows from S4B-PH-K to S5B-PH-K: GND_R / 5V / DRIVE / SENSE / CTRL.
- No-connect flags on D+/D-/SBU; ERC clean apart from the 'bridge' library
  path warnings. DRC: only the USB4085 footprint's inherent 0.15 mm
  pad-to-pad gaps and the edge-clipped silk at the receptacle remain.
- Title blocks, sheet notes and bottom silk at rev 0.6 / 2026-09-24.
- BOM: 13 Mouser line items; the rev 0.5 gerber zip is kept alongside.
Parts:
- added F1: 1.5A PTC, Fuse:Fuse_1812_4532Metric, symbol Device:Polyfuse
- added J3: USB4085 PWR, Connector_USB:USB_C_Receptacle_GCT_USB4085, symbol Connector:USB_C_Receptacle_USB2.0_16P
- added R10, R9: 5k1, Resistor_SMD:R_1206_3216Metric, symbol bridge:R_H
- J1: value APOLLO (P4 header GND,52,51,50) -> APOLLO (P4 header); footprint Connector_JST:JST_PH_S4B-PH-K_1x04_P2.00mm_Horizontal -> Connector_JST:JST_PH_S5B-PH-K_1x05_P2.00mm_Horizontal
- J2: value MACHINE: paddle pair + Micra white/black -> Micra: paddle tap
Connections:
- net CTRL: now also J1.5; no longer J1.4
- net DRIVE: now also J1.3; no longer J1.2
- net GND_R: now also J3.A1 (GND), J3.A12 (GND), J3.B1 (GND), J3.B12 (GND), J3.SH (SHIELD), R10.2, R9.2
- net SENSE: now also J1.4; no longer J1.3
- new net: J3.A5 (CC1), R9.1
- new net: J3.B5 (CC2), R10.1
- new net 5V: F1.2, J1.2
- new net VBUS: F1.1, J3.A4 (VBUS), J3.A9 (VBUS), J3.B4 (VBUS), J3.B9 (VBUS)
- no-connect marks 0 -> 6
Other:
- note added: "APOLLO PADDLE BRIDGE - rev 0.6 (2026-09-24)"
- note added: "Goal: unplug the remote and the Micra's paddle works as stock. The USB-C 5 V (J3) only passes through F1 (1.5 A PTC) to the remote on J1; every LED is still driven straight from a remote GPIO. CTRL (GPIO50) low or floating -> U2/U3 NC switches closed (paddle wired to the Micra in copper), NO switches open, remote fully disconnected. CTRL high (firmware, Wired paddle on) -> NC open, NO closed: pad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"
- note removed: "APOLLO PADDLE BRIDGE - rev 0.5 starting point (2026-09-16)"
- note removed: "Goal: unplug the remote and the Micra's paddle works as stock. No rail on this board: every LED is driven straight from a remote GPIO. CTRL (GPIO50) low or floating -> U2/U3 NC switches closed (paddle wired to the Micra in copper), NO switches open, remote fully disconnected. CTRL high (firmware, Wired paddle on) -> NC open, NO closed: paddle reads on SENSE (GPIO51), U1 alone drives the Micra fro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"
